File: DirtyNachos.kicad_sch (KiCad schematic)
At the start: 47 parts, among them J0 EURO_PWR_2x5, J1 OUTPUT, J2 INPUT, J3 CV IN, P1 Conn_01x01_Pin, P10 Conn_01x01_Pin, P10F1 Conn_01x01_Socket, P1F1 Conn_01x01_Socket, P2 Conn_01x01_Pin, P2F1 Conn_01x01_Socket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

Commit message: V0.2
More updates better paths ensuring aligment.
Other:
- title: (none) -> Schematics
Changed lines of the file:
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@@
 	(generator_version "8.0")
 	(paper "A4")
+	(title_block
+		(title "Schematics")
+		(date "2024-09-10")
+		(rev "0.2")
+	)
 	(junction
 		(at 63.5 144.78)
@@
 	(text "BIAS"
 		(exclude_from_sim no)
-		(at 102.616 68.072 0)
+		(at 102.87 68.58 0)
 		(effects
 			(font
@@
 	(text "CUTOFF"
 		(exclude_from_sim no)
-		(at 105.41 28.194 0)
+		(at 105.41 27.94 0)
 		(effects
 			(font
