File: DirtyNachos.kicad_pcb (KiCad board)
At the start: 2 copper layers, 78.5 x 107.5 mm, 49 parts, among them J0 EURO_PWR_2x5, J1 OUTPUT, J2 INPUT, J3 CV IN, P1 Conn_01x01_Pin, P10 Conn_01x01_Pin, P10F1 Conn_01x01_Socket, P1F1 Conn_01x01_Socket, P2 Conn_01x01_Pin, P2F1 Conn_01x01_Socket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

Commit message: Small updates.
Routing:
- net VCC: track 167.3 -> 3.21 mm, vias 2 -> 0
- net Net-(P4F1-Pin_1): track 103.6 -> 0.00 mm
- net Net-(P5-Pin_1): track 67.2 -> 0.00 mm
- net Net-(P7-Pin_1): track 54.5 -> 0.00 mm
- net Net-(P10F1-Pin_1): track 60.6 -> 11.1 mm, vias 1 -> 0
- net Net-(P1F1-Pin_1): track 48.3 -> 2.50 mm
- net Net-(P5F1-Pin_1): track 48.3 -> 2.79 mm, vias 2 -> 0
- net Net-(Q2-E): track 47.7 -> 4.53 mm, vias 1 -> 0
- net Net-(U1B--): track 46.5 -> 3.41 mm, vias 2 -> 0
- net Net-(P3F1-Pin_1): track 51.6 -> 8.82 mm
- net Net-(Q1-B): track 61.2 -> 19.4 mm, vias 2 -> 0
- net Net-(C3-Pad1): track 33.0 -> 6.33 mm
- net Net-(U1A--): track 26.4 -> 0.00 mm
- net Net-(P10-Pin_1): track 40.6 -> 14.4 mm
- net Net-(P7F1-Pin_1): track 30.9 -> 4.69 mm, vias 1 -> 0
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